File: hardware/electronics/electronics/_restore_backup_2026-08-18T23-50-42-462/electronics.kicad_pcb (KiCad board)
At the start: 2 copper layers, 130 x 100 mm, 14 parts, among them J1 Conn_Coaxial_Small, M1 Parachute_Servo, M2 Parachute_Servo, Q1 BC547, SW1 RBF, U1 RFM95W-915S2, U2 BMP585, U3 LSM6DS3, U4 SD Card mini module, U5 ESP32-S3-DEVKITC-1-N8R2, U6 GPS M8N, U7 MINI 560 STEP DOWN

Commit message: Update flight-computer hardware files
Parts:
- removed U3: LSM6DS3, electronics:LSM6DS3
- removed U6: GPS M8N, electronics:GPS N8M
- removed U7: MINI 560 STEP DOWN, electronics:STEP DOWN MINI 560
- moved J1 86.8 mm to (97.4, 119.0), turned to 0 degrees
- moved M1 82.4 mm to (272.1, 89.0)
- moved M2 79.0 mm to (276.7, 89.0)
- moved U1 77.4 mm to (93.7, 95.7), turned to 0 degrees
- moved U4 65.8 mm to (100.4, 85.7), turned to 180 degrees
- moved BZ1 45.9 mm to (156.0, 138.8)
- moved R1 45.9 mm to (146.5, 128.8)
- moved Q1 45.9 mm to (139.2, 134.3)
- moved SW1 18.5 mm to (254.6, 83.0)
- moved U2 17.2 mm to (143.1, 60.2)
Connections:
- M1 pad 2: /5 VCC -> /5 VCC SERVO
- M2 pad 2: /5 VCC -> /5 VCC SERVO
Routing:
- net /TX_GPS: track 90.5 -> 0.00 mm
- net /RX_GPS: track 78.8 -> 0.00 mm
- net /SCL: track 52.9 -> 0.00 mm
- net /3.3 VCC: track 70.5 -> 18.8 mm
- net /CS_SD: track 50.7 -> 0.00 mm
- net /5 VCC: track 46.4 -> 0.00 mm
- net /SDA: track 34.9 -> 0.00 mm
- net /SERVO: track 8.50 -> 0.00 mm
- net /LORA_DIO0: track 6.52 -> 0.00 mm
